Commit message: Adds KUKA iiwa 7 URDF

File: robots/iiwa7.urdf (robot description, URDF)
Before this commit: robot iiwa14, 10 links, 9 joints
Links:
- link iiwa_link_0: geometry collision mesh filename=package://iiwa_description/meshes/iiwa7/collision/link_0.stl; visual mesh filename=package://iiwa_description/meshes/iiwa7/visual/link_0.stl
- link iiwa_link_1: mass 4 -> 3.4525; geometry collision mesh filename=package://iiwa_description/meshes/iiwa7/collision/link_1.stl; visual mesh filename=package://iiwa_description/meshes/iiwa7/visual/link_1.stl
- link iiwa_link_2: mass 4 -> 3.4821; geometry collision mesh filename=package://iiwa_description/meshes/iiwa7/collision/link_2.stl; visual mesh filename=package://iiwa_description/meshes/iiwa7/visual/link_2.stl
- link iiwa_link_3: mass 3 -> 4.05623; geometry collision mesh filename=package://iiwa_description/meshes/iiwa7/collision/link_3.stl; visual mesh filename=package://iiwa_description/meshes/iiwa7/visual/link_3.stl
- link iiwa_link_4: mass 2.7 -> 3.4822; geometry collision mesh filename=package://iiwa_description/meshes/iiwa7/collision/link_4.stl; visual mesh filename=package://iiwa_description/meshes/iiwa7/visual/link_4.stl
- link iiwa_link_5: mass 1.7 -> 2.1633; geometry collision mesh filename=package://iiwa_description/meshes/iiwa7/collision/link_5.stl; visual mesh filename=package://iiwa_description/meshes/iiwa7/visual/link_5.stl
- link iiwa_link_6: mass 1.8 -> 2.3466; geometry collision mesh filename=package://iiwa_description/meshes/iiwa7/collision/link_6.stl; visual mesh filename=package://iiwa_description/meshes/iiwa7/visual/link_6.stl
- link iiwa_link_7: mass 0.3 -> 3.129; geometry collision mesh filename=package://iiwa_description/meshes/iiwa7/collision/link_7.stl; visual mesh filename=package://iiwa_description/meshes/iiwa7/visual/link_7.stl
Joints:
- joint iiwa_joint_1: origin xyz=0 0 0.1575 rpy=0 0 0 -> xyz=0 0 0.15 rpy=0 0 0
- joint iiwa_joint_2: origin xyz=0 0 0.2025 rpy=1.5707963267948966   0 3.141592653589793 -> xyz=0 0 0.19 rpy=1.5707963267948966   0 3.141592653589793
- joint iiwa_joint_3: origin xyz=0 0.2045 0 rpy=1.5707963267948966 0 3.141592653589793 -> xyz=0 0.21 0 rpy=1.5707963267948966 0 3.141592653589793
- joint iiwa_joint_4: origin xyz=0 0 0.2155 rpy=1.5707963267948966 0 0 -> xyz=0 0 0.19 rpy=1.5707963267948966 0 0
- joint iiwa_joint_5: origin xyz=0 0.1845 0 rpy=-1.5707963267948966 3.141592653589793 0 -> xyz=0 0.21 0 rpy=-1.5707963267948966 3.141592653589793 0
- joint iiwa_joint_6: origin xyz=0 0 0.2155 rpy=1.5707963267948966 0 0 -> xyz=0 0.06070 0.19 rpy=1.5707963267948966 0 0
- joint iiwa_joint_7: origin xyz=0 0.081 0 rpy=-1.5707963267948966 3.141592653589793 0 -> xyz=0 0.081 0.06070 rpy=-1.5707963267948966 3.141592653589793 0
