Commit message: Fixes Robotiq gripper finger joints

File: robots/gen3_robotiq_2f_140.urdf (robot description, URDF)
Before this commit: robot gen3_robotiq_2f_140, 24 links, 23 joints
Joints:
- joint finger_joint: type revolute -> fixed
- joint left_inner_finger_joint: type revolute -> fixed
- joint left_inner_knuckle_joint: type revolute -> fixed
- joint right_inner_finger_joint: type revolute -> fixed
- joint right_inner_knuckle_joint: type revolute -> fixed
- joint right_outer_knuckle_joint: type revolute -> fixed

File: robots/gen3_robotiq_2f_85.urdf (robot description, URDF)
Before this commit: robot gen3_robotiq_2f_85, 24 links, 23 joints
Joints:
- joint finger_joint: type revolute -> fixed
- joint left_inner_finger_joint: type revolute -> fixed
- joint left_inner_knuckle_joint: type revolute -> fixed
- joint right_inner_finger_joint: type revolute -> fixed
- joint right_inner_knuckle_joint: type revolute -> fixed
- joint right_outer_knuckle_joint: type revolute -> fixed
